File: adb_keyboard_converter/adb_converter.brd (EAGLE design)
At the start: 44.5 x 27.9 mm, 17 parts

Commit message: finish adb converter design
Parts:
- removed D1: GREEN, SparkFun-LED:LED-0603
- removed R5: 220, SparkFun-Resistors:0603-RES
- moved C2 6.82 mm to (17.3, 15.2), flipped to the bottom, turned to 180 degrees
- moved R6 4.54 mm to (13.0, 20.8), turned to 270 degrees
- moved D2 2.17 mm to (11.4, 20.8), turned to 180 degrees
- moved C1 1.09 mm to (18.8, 21.6), turned to 0 degrees
- moved JP2 0.76 mm to (7.62, 3.30)
- moved R3 0.76 mm to (15.2, 4.19)
Connections:
- removed net N$8: D1.C, R5.2
- removed net UVCC: JP1.VBUS, U$1.2, U$1.7
- net GND: no longer R5.1
- net STAT: no longer D1.A
- net VCC: now also JP1.VBUS, U$1.2, U$1.7
Routing:
- net STAT: track 18.4 -> 0.00 mm, vias 2 -> 0
- net SCK: track 0.00 -> 14.1 mm, vias 0 -> 1
- net MISO: track 0.00 -> 11.6 mm
- net MOSI: track 0.00 -> 8.48 mm
- net N$5: track 0.00 -> 3.30 mm, vias 0 -> 1
- net N$8: track 1.57 -> 0.00 mm
- net GND: track 25.9 -> 27.4 mm, vias 5 -> 7
- net N$3: track 9.72 -> 9.11 mm
