File: adb_keyboard_converter/adb_converter.sch (EAGLE design)
At the start: 17 parts

Commit message: finish adb converter design
Parts:
- removed D1: GREEN, SparkFun-LED:LED-GREEN0603
- removed R5: 220, SparkFun-Resistors:220OHM-1/10W-1%(0603)
Connections:
- removed net N$8: D1.C, R5.2
- removed net UVCC: JP1.VBUS, U$1.UVCC, U$1.VBUS
- net GND: no longer R5.1
- net STAT: no longer D1.A
- net VCC: now also JP1.VBUS, U$1.UVCC, U$1.VBUS
Other:
- moved on the sheet: D2, R6
Changed lines of the file:
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@@
 <part name="C4" library="SparkFun-Capacitors" deviceset="22PF-50V-5%(0603)" device="" value="22pF"/>
 <part name="GND7" library="SparkFun-Aesthetics" deviceset="GND" device=""/>
-<part name="D1" library="SparkFun-LED" deviceset="LED-GREEN" device="0603" value="GREEN"/>
 <part name="D2" library="SparkFun-LED" deviceset="LED-BLUE" device="0603" value="BLUE"/>
 <part name="GND8" library="SparkFun-Aesthetics" deviceset="GND" device=""/>
 <part name="SUPPLY6" library="SparkFun-Aesthetics" deviceset="VCC" device=""/>
-<part name="R5" library="SparkFun-Resistors" deviceset="220OHM-1/10W-1%(0603)" device="" value="220"/>
 <part name="R6" library="SparkFun-Resistors" deviceset="220OHM-1/10W-1%(0603)" device="" value="220"/>
+<part name="SUPPLY7" library="SparkFun-Aesthetics" deviceset="VCC" device=""/>
+<part name="SUPPLY8" library="SparkFun-Aesthetics" deviceset="VCC" device=""/>
 </parts>
 <sheets>
@@
 <instance part="C4" gate="G$1" x="71.12" y="30.48" rot="R90"/>
 <instance part="GND7" gate="1" x="58.42" y="33.02" rot="R270"/>
-<instance part="D1" gate="G$1" x="17.78" y="48.26"/>
-<instance part="D2" gate="G$1" x="27.94" y="48.26"/>
+<instance part="D2" gate="G$1" x="22.86" y="48.26"/>
 <instance part="GND8" gate="1" x="22.86" y="25.4"/>
-<instance part="SUPPLY6" gate="G$1" x="27.94" y="53.34"/>
-<instance part="R5" gate="G$1" x="17.78" y="38.1" rot="R90"/>
-<instance part="R6" gate="G$1" x="27.94" y="38.1" rot="R90"/>
+<instance part="SUPPLY6" gate="G$1" x="22.86" y="53.34"/>
+<instance part="R6" gate="G$1" x="22.86" y="35.56" rot="R90"/>
+<instance part="SUPPLY7" gate="G$1" x="83.82" y="60.96"/>
+<instance part="SUPPLY8" gate="G$1" x="55.88" y="20.32"/>
 </instances>
 <busses>
@@
 </segment>
 <segment>
-<pinref part="R5" gate="G$1" pin="1"/>
-<wire x1="17.78" y1="33.02" x2="17.78" y2="30.48" width="0.1524" layer="91"/>
-<pinref part="R6" gate="G$1" pin="1"/>
-<wire x1="17.78" y1="30.48" x2="22.86" y2="30.48" width="0.1524" layer="91"/>
-<wire x1="22.86" y1="30.48" x2="27.94" y2="30.48" width="0.1524" layer="91"/>
-<wire x1="27.94" y1="30.48" x2="27.94" y2="33.02" width="0.1524" layer="91"/>
 <pinref part="GND8" gate="1" pin="GND"/>
 <wire x1="22.86" y1="27.94" x2="22.86" y2="30.48" width="0.1524" layer="91"/>
-<junction x="22.86" y="30.48"/>
+<pinref part="R6" gate="G$1" pin="1"/>
 </segment>
 </net>
@@
 <wire x1="45.72" y1="12.7" x2="50.8" y2="12.7" width="0.1524" layer="91"/>
 <pinref part="R2" gate="G$1" pin="1"/>
-</segment>
-</net>
-<net name="UVCC" class="0">
-<segment>
-<pinref part="JP1" gate="G$1" pin="VBUS"/>
-<wire x1="45.72" y1="17.78" x2="55.88" y2="17.78" width="0.1524" layer="91"/>
-<label x="53.34" y="17.78" size="1.27" layer="95"/>
-</segment>
-<segment>
-<pinref part="U$1" gate="G$1" pin="UVCC"/>
-<wire x1="86.36" y1="55.88" x2="83.82" y2="55.88" width="0.1524" layer="91"/>
-<wire x1="83.82" y1="55.88" x2="83.82" y2="58.42" width="0.1524" layer="91"/>
-<pinref part="U$1" gate="G$1" pin="VBUS"/>
-<wire x1="83.82" y1="58.42" x2="83.82" y2="60.96" width="0.1524" layer="91"/>
-<wire x1="86.36" y1="58.42" x2="83.82" y2="58.42" width="0.1524" layer="91"/>
-<junction x="83.82" y="58.42"/>
-<wire x1="83.82" y1="60.96" x2="78.74" y2="60.96" width="0.1524" layer="91"/>
-<label x="78.74" y="60.96" size="1.27" layer="95"/>
 </segment>
 </net>
@@
 <pinref part="D2" gate="G$1" pin="A"/>
 <pinref part="SUPPLY6" gate="G$1" pin="VCC"/>
-<wire x1="27.94" y1="50.8" x2="27.94" y2="53.34" width="0.1524" layer="91"/>
+<wire x1="22.86" y1="50.8" x2="22.86" y2="53.34" width="0.1524" layer="91"/>
+</segment>
+<segment>
+<pinref part="JP1" gate="G$1" pin="VBUS"/>
+<wire x1="45.72" y1="17.78" x2="55.88" y2="17.78" width="0.1524" layer="91"/>
+<wire x1="55.88" y1="17.78" x2="55.88" y2="20.32" width="0.1524" layer="91"/>
+<pinref part="SUPPLY8" gate="G$1" pin="VCC"/>
+</segment>
+<segment>
+<pinref part="U$1" gate="G$1" pin="UVCC"/>
+<wire x1="86.36" y1="55.88" x2="83.82" y2="55.88" width="0.1524" layer="91"/>
+<wire x1="83.82" y1="55.88" x2="83.82" y2="58.42" width="0.1524" layer="91"/>
+<pinref part="U$1" gate="G$1" pin="VBUS"/>
+<wire x1="83.82" y1="58.42" x2="83.82" y2="60.96" width="0.1524" layer="91"/>
+<wire x1="86.36" y1="58.42" x2="83.82" y2="58.42" width="0.1524" layer="91"/>
+<junction x="83.82" y="58.42"/>
+<pinref part="SUPPLY7" gate="G$1" pin="VCC"/>
 </segment>
 </net>
@@
 <label x="129.54" y="25.4" size="1.27" layer="95"/>
 </segment>
-<segment>
-<pinref part="D1" gate="G$1" pin="A"/>
-<wire x1="17.78" y1="50.8" x2="17.78" y2="53.34" width="0.1524" layer="91"/>
-<wire x1="17.78" y1="53.34" x2="22.86" y2="53.34" width="0.1524" layer="91"/>
-<label x="20.32" y="53.34" size="1.27" layer="95"/>
-</segment>
-</net>
-<net name="N$8" class="0">
-<segment>
-<pinref part="D1" gate="G$1" pin="C"/>
-<pinref part="R5" gate="G$1" pin="2"/>
-</segment>
 </net>
 <net name="N$9" class="0">
@@
 <pinref part="D2" gate="G$1" pin="C"/>
 <pinref part="R6" gate="G$1" pin="2"/>
-</segment>
-</net>
+<wire x1="22.86" y1="40.64" x2="22.86" y2="43.18" width="0.1524" layer="91"/>
+</segment>
+</net>
